File: module/SMTRelayControllerDense.brd (EAGLE design)
At the start: 56.8 x 64.8 mm, 38 parts, among them T2 MMBT3904, T3 MMBT3904, T4 MMBT3906, T7 MMBT3904, U1 L298

Commit message: saved dense schematic
Parts:
- removed LOGO1: OSHW-LOGOM-COPPER, SparkFun-Aesthetics:OSHW-LOGO-M_COPPER
- added LOGO2: OSHW-LOGOM, SparkFun-Aesthetics:OSHW-LOGO-M
- moved JP4 42.4 mm to (52.3, 14.0), turned to 270 degrees
- moved C3 28.9 mm to (45.7, 13.0), turned to 270 degrees
- moved R3 11.4 mm to (15.5, 26.7), turned to 270 degrees
- moved C2 11.4 mm to (13.7, 16.5)
- moved C4 11.4 mm to (16.3, 39.4)
- moved C5 11.4 mm to (21.3, 39.4)
- moved D1 11.4 mm to (13.7, 8.89)
- moved D4 11.4 mm to (45.5, 40.6)
- moved D5 11.4 mm to (45.5, 45.7)
- moved D6 11.4 mm to (9.91, 31.8)
- moved D8 11.4 mm to (39.1, 40.6)
- moved D9 11.4 mm to (39.1, 45.7)
- moved JP1 11.4 mm to (22.6, 45.7)
- moved JP2 11.4 mm to (11.2, 45.7)
- moved JP6 11.4 mm to (51.8, 35.6)
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Routing:
- net VCC: track 105.1 -> 140.7 mm, vias 6 -> 3
- net V_RAW: track 122.0 -> 156.9 mm
- net RELAY_ENA: track 65.2 -> 89.3 mm, vias 3 -> 0
- net GND: track 108.8 -> 91.5 mm
- net TX_SENSE_IN: track 68.4 -> 58.3 mm
- net RX_CTL: track 55.9 -> 52.0 mm, vias 0 -> 3
- net RX_SENSE_IN: track 49.5 -> 53.2 mm
- net PTT_L: track 47.0 -> 43.8 mm
- net V_IN: track 30.8 -> 33.4 mm
- net TX_CTL: track 66.7 -> 65.0 mm, vias 0 -> 2
- net N$6: track 3.43 -> 2.16 mm
- net N$3: track 3.43 -> 2.16 mm
Other:
- board size 56.8 x 64.8 mm -> 56.8 x 53.3 mm
- board text added: "2016"
- board text added: "CC BY-SA 4.0"
- board text added: "CC-BY-SA"
- board text added: "KB1VC Relay Controller Module"
- board text added: "M. H. Reilly"
- board text added: "RF Relay Controller"
- board text added: "Rev B Oct 2016"
- board text added: "Rev B_SMT"
- board text added: "See the license file at https://creativecommons.org/licenses/by-sa/4.0/"
- board text added: "https://github.com/kb1vc/RelayControl"
