File: module/SMTRelayControllerDense.sch (EAGLE design)
At the start: 38 parts, among them T2 MMBT3904, T3 MMBT3904, T4 MMBT3906, T7 MMBT3904, U1 L298

Commit message: saved dense schematic
Parts:
- removed LOGO1: OSHW-LOGOM-COPPER, SparkFun-Aesthetics:OSHW-LOGOM-COPPER
- added LOGO2: OSHW-LOGOM, SparkFun-Aesthetics:OSHW-LOGOM
Changed lines of the file:
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@@
 <part name="R9" library="rcl" deviceset="R-US_" device="R1206" value="10K"/>
 <part name="R10" library="rcl" deviceset="R-US_" device="R1206" value="10K"/>
-<part name="LOGO1" library="SparkFun-Aesthetics" deviceset="OSHW-LOGO" device="M-COPPER"/>
 <part name="T2" library="transistor-neu-to92" deviceset="*-NPN-" device="SOT23-BEC" technology="MMBT3904LT1" value="MMBT3904"/>
 <part name="D3" library="SparkFun-LED" deviceset="LED" device="1206" value="GREEN"/>
@@
 <part name="R11" library="rcl" deviceset="R-US_" device="R1206" value="10K"/>
 <part name="C3" library="resistor" deviceset="C-US" device="C1206K" value="0.15"/>
+<part name="LOGO2" library="SparkFun-Aesthetics" deviceset="OSHW-LOGO" device="M"/>
 </parts>
 <sheets>
@@
 <instance part="R9" gate="G$1" x="-236.22" y="30.48"/>
 <instance part="R10" gate="G$1" x="-187.96" y="30.48"/>
-<instance part="LOGO1" gate="G$1" x="-248.92" y="210.82"/>
 <instance part="T2" gate="G$1" x="-226.06" y="30.48" smashed="yes">
 <attribute name="NAME" x="-220.98" y="30.48" size="1.778" layer="95"/>
@@
 <instance part="R11" gate="G$1" x="-226.06" y="127"/>
 <instance part="C3" gate="G$1" x="-124.46" y="162.56"/>
+<instance part="LOGO2" gate="G$1" x="-248.92" y="208.28"/>
 </instances>
 <busses>
